File: board/SkyMusicPad.kicad_sch (KiCad schematic)
At the start: 36 parts, among them SW1 Cherry, SW10 Cherry, SW11 Cherry, SW12 Cherry, SW13 Cherry, SW14 Cherry, SW15 Cherry, SW16 RotaryEncoder_Switch, SW2 Cherry, SW3 Cherry, SW4 Cherry, SW5 Cherry, SW6 Cherry, SW7 Cherry, SW8 Cherry, SW9 Cherry

Commit message: i hate this
Parts:
- removed RZ1: RP2040-Zero, RP2040-Zero:RP2040-Zero, symbol rp2040-zero:RP2040-Zero
- added D16, D17, D18, D19, D20, D21, D22, D23, D24, D25, D26, D27, D28, D29, D30: SK6812MINI, SkyMusic:LED_SK6812MINI_REVERSE, symbol LED:SK6812MINI
- added U1: ESP32-S3-Zero, ESP32-S3-Zero:ESP32-S3-Zero, symbol ESP32-S3-Zero:ESP32-S3-Zero
Connections:
- net +3.3V: now also D16.4 (VDD), D17.4 (VDD), D18.4 (VDD), D19.4 (VDD), D20.4 (VDD), D21.4 (VDD), D22.4 (VDD), D23.4 (VDD), D24.4 (VDD), D25.4 (VDD), D26.4 (VDD), D27.4 (VDD), D28.4 (VDD), D29.4 (VDD), D30.4 (VDD), U1.16 (3V3)
- net +5V: now also U1.18 (5V)
- net Col0: now also U1.11 (GP5)
- net Col1: now also U1.12 (GP4)
- net Col2: now also U1.13 (GP3)
- net Col3: now also U1.14 (GP2)
- net Col4: now also U1.15 (GP1)
- net GND: now also D16.2 (VSS), D17.2 (VSS), D18.2 (VSS), D19.2 (VSS), D20.2 (VSS), D21.2 (VSS), D22.2 (VSS), D23.2 (VSS), D24.2 (VSS), D25.2 (VSS), D26.2 (VSS), D27.2 (VSS), D28.2 (VSS), D29.2 (VSS), D30.2 (VSS), U1.17 (GND)
- net Rot_A: now also U1.6 (GP10)
- net Rot_B: now also U1.7 (GP9)
- net Rot_SW: now also U1.2 (RX)
- net Row0: now also U1.8 (GP8)
- net Row1: now also U1.9 (GP7)
- net Row2: now also U1.10 (GP6)
- new net: D29.1 (DOUT), D30.3 (DIN)
- new net: D28.1 (DOUT), D29.3 (DIN)
- new net: D24.1 (DOUT), D25.3 (DIN)
- new net: D23.1 (DOUT), D24.3 (DIN)
- new net: D18.1 (DOUT), D19.3 (DIN)
- new net: D17.1 (DOUT), D18.3 (DIN)
- new net: D16.1 (DOUT), D17.3 (DIN)
- new net: D22.1 (DOUT), D23.3 (DIN)
- new net: D21.1 (DOUT), D22.3 (DIN)
- new net: D19.1 (DOUT), D20.3 (DIN)
- new net: D26.1 (DOUT), D27.3 (DIN)
- new net: D27.1 (DOUT), D28.3 (DIN)
- new net Neopixel: D16.3 (DIN), U1.5 (GP11)
- new net Row0_out: D20.1 (DOUT), D21.3 (DIN)
- new net Row1_out: D25.1 (DOUT), D26.3 (DIN)
- new net SCL: U1.4 (GP12)
- new net SDA: U1.3 (GP13)
Other:
- moved on the sheet: D1, D10, D11, D12, D13, D14, D15, D2, D3, D4, D5, D6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

Commit message: Fix minor issues, adjust diode silkscreen
Parts:
- D1, D10, D11, D12, D13, D14, D15, D2, D3, D4, D5, D6, D7, D8, D9: footprint Diode_SMD:D_MiniMELF -> SkyMusic:D_MiniMELF_silkMoved
Changed lines of the file:
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@@
 			)
 		)
-		(property "Footprint" "Diode_SMD:D_MiniMELF"
+		(property "Footprint" "SkyMusic:D_MiniMELF_silkMoved"
 			(at 121.92 59.69 90)
 			(effects
@@
 			)
 		)
-		(property "Footprint" "Diode_SMD:D_MiniMELF"
+		(property "Footprint" "SkyMusic:D_MiniMELF_silkMoved"
 			(at 59.69 71.12 90)
 			(effects
@@
 			)
 		)
-		(property "Footprint" "Diode_SMD:D_MiniMELF"
+		(property "Footprint" "SkyMusic:D_MiniMELF_silkMoved"
 			(at 121.92 71.12 90)
 			(effects
@@
 			)
 		)
-		(property "Footprint" "Diode_SMD:D_MiniMELF"
+		(property "Footprint" "SkyMusic:D_MiniMELF_silkMoved"
 			(at 100.33 71.12 90)
 			(effects
@@
 			)
 		)
-		(property "Footprint" "Diode_SMD:D_MiniMELF"
+		(property "Footprint" "SkyMusic:D_MiniMELF_silkMoved"
 			(at 80.01 71.12 90)
 			(effects
@@
 			)
 		)
-		(property "Footprint" "Diode_SMD:D_MiniMELF"
+		(property "Footprint" "SkyMusic:D_MiniMELF_silkMoved"
 			(at 39.37 59.69 90)
 			(effects
@@
 			)
 		)
-		(property "Footprint" "Diode_SMD:D_MiniMELF"
+		(property "Footprint" "SkyMusic:D_MiniMELF_silkMoved"
 			(at 39.37 48.26 90)
 			(effects
@@
 			)
 		)
-		(property "Footprint" "Diode_SMD:D_MiniMELF"
+		(property "Footprint" "SkyMusic:D_MiniMELF_silkMoved"
 			(at 80.01 59.69 90)
 			(effects
@@
 			)
 		)
-		(property "Footprint" "Diode_SMD:D_MiniMELF"
+		(property "Footprint" "SkyMusic:D_MiniMELF_silkMoved"
 			(at 100.33 59.69 90)
 			(effects
@@
 			)
 		)
-		(property "Footprint" "Diode_SMD:D_MiniMELF"
+		(property "Footprint" "SkyMusic:D_MiniMELF_silkMoved"
 			(at 59.69 48.26 90)
 			(effects
@@
 			)
 		)
-		(property "Footprint" "Diode_SMD:D_MiniMELF"
+		(property "Footprint" "SkyMusic:D_MiniMELF_silkMoved"
 			(at 80.01 48.26 90)
 			(effects
@@
 			)
 		)
-		(property "Footprint" "Diode_SMD:D_MiniMELF"
+		(property "Footprint" "SkyMusic:D_MiniMELF_silkMoved"
 			(at 59.69 59.69 90)
 			(effects
@@
 			)
 		)
-		(property "Footprint" "Diode_SMD:D_MiniMELF"
+		(property "Footprint" "SkyMusic:D_MiniMELF_silkMoved"
 			(at 121.92 48.26 90)
 			(effects
@@
 			)
 		)
-		(property "Footprint" "Diode_SMD:D_MiniMELF"
+		(property "Footprint" "SkyMusic:D_MiniMELF_silkMoved"
 			(at 39.37 71.12 90)
 			(effects
@@
 			)
 		)
-		(property "Footprint" "Diode_SMD:D_MiniMELF"
+		(property "Footprint" "SkyMusic:D_MiniMELF_silkMoved"
 			(at 100.33 48.26 90)
 			(effects

Commit message: Adjusted LED silk, need to fix encoder
Parts:
- SW16: footprint Rotary_Encoder:RotaryEncoder_Bourns_Vertical_PEC12R-3x17F-Sxxxx -> SkyMusic:RotaryEncoder_Bourns_Vertical_PEC12R-3x17F-Sxxxx
Changed lines of the file:
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@@
 			)
 		)
-		(property "Footprint" "Rotary_Encoder:RotaryEncoder_Bourns_Vertical_PEC12R-3x17F-Sxxxx"
+		(property "Footprint" "SkyMusic:RotaryEncoder_Bourns_Vertical_PEC12R-3x17F-Sxxxx"
 			(at 138.43 115.316 0)
 			(effects

Commit message: misc updates
Connections:
- net Rot_A: now also SW16.B; no longer SW16.A
- net Rot_B: now also SW16.A; no longer SW16.B
Changed lines of the file:
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@@
 	(global_label "Rot_A"
 		(shape bidirectional)
-		(at 130.81 116.84 180)
-		(fields_autoplaced yes)
-		(effects
-			(font
-				(size 1.27 1.27)
-			)
-			(justify right)
-		)
-		(property "Intersheetrefs" "${INTERSHEET_REFS}"
-			(at 121.5126 116.84 0)
+		(at 130.81 121.92 180)
+		(fields_autoplaced yes)
+		(effects
+			(font
+				(size 1.27 1.27)
+			)
+			(justify right)
+		)
+		(property "Intersheetrefs" "${INTERSHEET_REFS}"
+			(at 121.5126 121.92 0)
 			(effects
 				(font
@@
 	(global_label "Rot_B"
 		(shape bidirectional)
-		(at 130.81 121.92 180)
-		(fields_autoplaced yes)
-		(effects
-			(font
-				(size 1.27 1.27)
-			)
-			(justify right)
-		)
-		(property "Intersheetrefs" "${INTERSHEET_REFS}"
-			(at 121.3312 121.92 0)
-			(effects
-				(font
+		(at 130.81 116.84 180)
+		(fields_autoplaced yes)
+		(effects
+			(font
+				(size 1.27 1.27)
+			)
+			(justify right)
+		)
+		(property "Intersheetrefs" "${INTERSHEET_REFS}"
+			(at 121.3312 116.84 0)
+			(effects
+				(font

Commit message: Components placed
Parts:
- added J1: Conn_01x04, SkyMusic:OLED_DFR0648, symbol Connector_Generic:Conn_01x04
Connections:
- net +3.3V: now also U1.3 (3V3), J1.1 (Pin_1); no longer U1.16 (3V3)
- net +5V: now also U1.1 (5V); no longer U1.18 (5V)
- net Col0: now also U1.8 (GP5); no longer U1.11 (GP5)
- net Col1: now also U1.7 (GP4); no longer U1.12 (GP4)
- net Col2: now also U1.6 (GP3); no longer U1.13 (GP3)
- net Col3: now also U1.5 (GP2); no longer U1.14 (GP2)
- net Col4: now also U1.4 (GP1); no longer U1.15 (GP1)
- net GND: now also U1.2 (GND), J1.2 (Pin_2); no longer U1.17 (GND)
- net Neopixel: now also U1.11 (GP8); no longer U1.5 (GP11)
- net Rot_A: no longer U1.6 (GP10)
- net Rot_B: no longer U1.7 (GP9)
- net Rot_SW: no longer U1.2 (RX)
- net Row0: now also U1.14 (GP11); no longer U1.8 (GP8)
- net Row1: now also U1.13 (GP10); no longer U1.9 (GP7)
- net Row2: now also U1.12 (GP9); no longer U1.10 (GP6)
- net SCL: now also U1.16 (GP13), J1.3 (Pin_3); no longer U1.4 (GP12)
- net SDA: now also U1.15 (GP12), J1.4 (Pin_4); no longer U1.3 (GP13)

Commit message: Add charging circuit, finalising design
Parts:
- removed H4: GND, MountingHole:MountingHole_2.2mm_M2_Pad_Via, symbol Mechanical:MountingHole_Pad
- added BT1: Battery_Cell, Connector_JST:JST_PH_B2B-PH-K_1x02_P2.00mm_Vertical, symbol Device:Battery_Cell
- added C1: 1uF, Capacitor_SMD:C_0603_1608Metric, symbol Device:C_Small
- added C2, C5, C6: 10uF, Capacitor_SMD:C_0603_1608Metric, symbol Device:C_Small
- added C3: 47nF, Capacitor_SMD:C_0603_1608Metric, symbol Device:C_Small
- added C4: 4.7uF, Capacitor_SMD:C_0603_1608Metric, symbol Device:C_Small
- added C7: 40uF, Capacitor_SMD:C_0603_1608Metric, symbol Device:C_Small
- added L1: 2.2uH, Inductor_SMD:L_Vishay_IHLP-2020, symbol Device:L_Small
- added R1: 260, Resistor_SMD:R_0603_1608Metric, symbol Device:R_Small
- added R2: 30.1k, Resistor_SMD:R_0603_1608Metric, symbol Device:R_Small
- added R3: 5.23k, Resistor_SMD:R_0603_1608Metric, symbol Device:R_Small
- added U2: BQ25895RTW, Package_DFN_QFN:Texas_RTW_WQFN-24-1EP_4x4mm_P0.5mm_EP2.7x2.7mm_ThermalVias, symbol Battery_Management:BQ25895RTW
Connections:
- net +5V: now also C1.1, U2.1 (VBUS)
- net GND: now also BT1.2 (-), C1.2, C2.2, C4.1, C5.2, C6.2, C7.1, R1.1, R2.1, U2.17 (PGND), U2.18 (PGND), U2.25 (PGND), U2.9 (~{CE})
- net Neopixel: now also U1.13 (GP10); no longer U1.11 (GP8)
- net Rot_A: now also U1.20 (GP18)
- net Rot_B: now also U1.19 (GP17)
- net Rot_SW: now also U1.9 (GP6)
- net Row1: now also U1.12 (GP9); no longer U1.13 (GP10)
- net Row2: now also U1.11 (GP8); no longer U1.12 (GP9)
- net SCL: now also U2.5 (SCL)
- net SDA: now also U2.6 (SDA)
- new net: BT1.1 (+), C2.1, U2.13 (BAT), U2.14 (BAT)
- new net: R2.2, R3.1, U2.11 (TS)
- new net: C4.2, R3.2, U2.22 (REGN)
- new net: R1.2, U2.10 (ILIM)
- new net: C3.1, L1.1, U2.19 (SW), U2.20 (SW)
- new net: C3.2, U2.21 (BTST)
- new net: C7.2, U2.23 (PMID)
- new net BQ_STAT: U2.4 (STAT)
- new net VCC: C5.1, C6.1, L1.2, U2.15 (SYS), U2.16 (SYS)
- no-connect marks 0 -> 5

Commit message: Begin work on battery
Parts:
- removed BT1: Battery_Cell, Connector_JST:JST_PH_B2B-PH-K_1x02_P2.00mm_Vertical, symbol Device:Battery_Cell
- removed C1: 1uF, Capacitor_SMD:C_0603_1608Metric, symbol Device:C_Small
- removed C2, C5, C6: 10uF, Capacitor_SMD:C_0603_1608Metric, symbol Device:C_Small
- removed C3: 47nF, Capacitor_SMD:C_0603_1608Metric, symbol Device:C_Small
- removed C4: 4.7uF, Capacitor_SMD:C_0603_1608Metric, symbol Device:C_Small
- removed C7: 40uF, Capacitor_SMD:C_0603_1608Metric, symbol Device:C_Small
- removed L1: 2.2uH, Inductor_SMD:L_Vishay_IHLP-2020, symbol Device:L_Small
- removed R1: 260, Resistor_SMD:R_0603_1608Metric, symbol Device:R_Small
- removed R2: 30.1k, Resistor_SMD:R_0603_1608Metric, symbol Device:R_Small
- removed R3: 5.23k, Resistor_SMD:R_0603_1608Metric, symbol Device:R_Small
- removed U2: BQ25895RTW, Package_DFN_QFN:Texas_RTW_WQFN-24-1EP_4x4mm_P0.5mm_EP2.7x2.7mm_ThermalVias, symbol Battery_Management:BQ25895RTW
- added C8, C9: 10uF, Capacitor_SMD:C_0603_1608Metric, symbol Device:C_Small
- added J2: BatteryCharger, Connector_PinHeader_2.54mm:PinHeader_1x04_P2.54mm_Vertical, symbol Connector_Generic:Conn_01x04
- added U3: XC6220B331MR, Package_TO_SOT_SMD:SOT-23-5, symbol Regulator_Linear:XC6220B331MR
Connections:
- net +3.3V: now also C8.1, U3.5 (VOUT)
- net +5V: now also J2.3 (Pin_3)
- net GND: now also C8.2, C9.2, J2.4 (Pin_4), U3.2 (GND)
- net VCC: now also C9.1, J2.1 (Pin_1), U3.1 (VIN), U3.3 (CE)
- new net BATT: J2.2 (Pin_2)
- no-connect marks 5 -> 0

Commit message: Near completion, pretty much done I think
Parts:
- removed J2: BatteryCharger, Connector_PinHeader_2.54mm:PinHeader_1x04_P2.54mm_Vertical, symbol Connector_Generic:Conn_01x04
- added BT1: Battery_Cell, Connector_JST:JST_PH_B2B-PH-SM4-TB_1x02-1MP_P2.00mm_Vertical, symbol Device:Battery_Cell
- added C3, C4: 10uF, Capacitor_SMD:C_0603_1608Metric, symbol Device:C_Small
- added D31: D_Small, Diode_SMD:D_1206_3216Metric, symbol Device:D_Small
- added R1: 600, Resistor_SMD:R_0603_1608Metric, symbol Device:R_Small
- added SW17: SW_SPDT, SkyMusic:SSAJ120100, symbol Switch:SW_SPDT
- added U2: TP4056-42-ESOP8, Package_SO:SOIC-8-1EP_3.9x4.9mm_P1.27mm_EP2.41x3.3mm_ThermalVias, symbol Battery_Management:TP4056-42-ESOP8
- renumbered C9 to C1, C8 to C2
Connections:
- net +5V: now also C3.1, U2.4 (V_{CC}), U2.8 (CE)
- net BATT: now also BT1.1 (+), C4.1, D31.2 (A), U2.5 (BAT)
- net GND: now also BT1.2 (-), BT1.MP (-), C3.2, C4.2, R1.1, SW17.MP, U2.1 (TEMP), U2.3 (GND), U2.6 (~{STDBY}), U2.9 (EPAD)
- net VCC: now also SW17.2 (B)
- net CHRG: now reaches U1.25 (GP42)
- net CHRG: now also U2.7 (~{CHRG})
- new net: D31.1 (K), SW17.3 (A)
- new net: R1.2, U2.2 (PROG)
- no-connect marks 0 -> 1
Other:
- moved on the sheet: H1, H2, H3
